Commit message: refactor(dm_arm_description): 改用官方 urdf

File: src/dm_arm_description/urdf/DM-Arm-Description.urdf (robot description, URDF)
Before this commit: robot DM-Arm-Description, 12 links, 11 joints
Links:
- removed link base_footprint
- removed link link1
- removed link link2
- removed link link_tcp
- added link camera
- added link link2-3, mass 0.9084; collision mesh filename=package://dm_arm_description/meshes/collision/link2-3.stl; visual mesh filename=package://dm_arm_description/meshes/visual/link2-3.glb
- added link link3-4, mass 0.7089; collision mesh filename=package://dm_arm_description/meshes/collision/link3-4.stl; visual mesh filename=package://dm_arm_description/meshes/visual/link3-4.glb
- link base_link: mass None -> 0.5111; geometry collision mesh filename=package://dm_arm_description/meshes/collision/base_link.stl; visual mesh filename=package://dm_arm_description/meshes/visual/base_link.glb
- link finger_left: mass None -> 0.05; geometry collision mesh filename=package://dm_arm_description/meshes/collision/finger_left.s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; visual mesh filename=package://dm_arm_description/meshes/visual/finger_left.glb
- link finger_right: mass None -> 0.05; geometry collision mesh filename=package://dm_arm_description/meshes/collision/finger_right.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; visual mesh filename=package://dm_arm_description/meshes/visual/finger_right.glb
- link link1-2: mass None -> 0.5965; geometry collision mesh filename=package://dm_arm_description/meshes/collision/link1-2.stl; visual mesh filename=package://dm_arm_description/meshes/visual/link1-2.glb
- link link4-5: mass None -> 0.3995; geometry collision mesh filename=package://dm_arm_description/meshes/collision/link4-5.stl; visual mesh filename=package://dm_arm_description/meshes/visual/link4-5.glb
- link link5-6: mass None -> 0.4121; geometry collision mesh filename=package://dm_arm_description/meshes/collision/link5-6.stl; visual mesh filename=package://dm_arm_description/meshes/visual/link5-6.glb
- link link6-7: mass None -> 0.5; geometry collision mesh filename=package://dm_arm_description/meshes/collision/link6-7.stl; visual mesh filename=package://dm_arm_description/meshes/visual/link6-7.glb
Joints:
- removed joint base_footprint_joint
- removed joint joint_tcp
- added joint camera_joint: type fixed, parent link6-7, child camera, origin xyz=0.0471 0 0.063314 rpy=0 0.2618 0
- joint gripper_left: axis -1 0 0 -> 0 1 0; limit lower=-0.045 upper=0.0 effort=20 velocity=0.2 -> lower=-0.045 upper=0.001 effort=20 velocity=0.18
- joint gripper_right: axis 1 0 0 -> 0 -1 0; limit lower=-0.045 upper=0.0 effort=20 velocity=0.2 -> lower=-0.045 upper=0.001 effort=20 velocity=0.18; mimic joint=gripper_left multiplier=1 offset=0 -> (none)
- joint gripper_tool0: origin xyz=0 0.158 0 rpy=-1.5707963267948966 0 0 -> xyz=0.158 0 0 rpy=-1.5707963267948966 0 -1.5707963267948966
- joint joint1: limit lower=-2.0943951023931953 upper=2.0943951023931953 effort=100 velocity=3 -> lower=-2.0943951023931953 upper=2.0943951023931953 effort=100 velocity=5.4
- joint joint2: axis -1 0 0 -> 0 1 0; child link1 -> link2-3; limit lower=0.0 upper=3.141592653589793 effort=100 velocity=3 -> lower=-0.01 upper=3.141592653589793 effort=100 velocity=5.4; origin xyz=0 0.02 0.0385 rpy=0 0 0 -> xyz=0.02 0.0 0.0385 rpy=0 0 0
- joint joint3: axis 1 0 0 -> 0 -1 0; child link2 -> link3-4; limit lower=0.0 upper=4.71238898038469 effort=100 velocity=3 -> lower=-0.01 upper=4.71238898038469 effort=100 velocity=5.4; origin xyz=0 -0.264 0 rpy=0 0 0 -> xyz=-0.264 0 0 rpy=0 0 0; parent link1 -> link2-3
- joint joint4: axis 1 0 0 -> 0 -1 0; limit lower=-1.5707963267948966 upper=1.5707963267948966 effort=20 velocity=3 -> lower=-1.95 upper=1.5707963267948966 effort=20 velocity=5.4; origin xyz=0 0.244004 0.059971 rpy=0 0 0 -> xyz=0.244004 0 0.059971 rpy=0 0 0; parent link2 -> link3-4
- joint joint5: limit lower=-1.5707963267948966 upper=1.5707963267948966 effort=20 velocity=3 -> lower=-1.5707963267948966 upper=1.5707963267948966 effort=20 velocity=5.4; origin xyz=0 0.061868 0.0425 rpy=0 0 0 -> xyz=0.061868 0 0.0425 rpy=0 0 0
- joint joint6: axis 0 1 0 -> 1 0 0; limit lower=-3.141592653589793 upper=3.141592653589793 effort=20 velocity=3 -> lower=-3.141592653589793 upper=3.141592653589793 effort=20 velocity=5.4; origin xyz=0.0 0.032 -0.0425 rpy=0 0 0 -> xyz=0.032 0 -0.0425 rpy=0 0 0

Commit message: feat(dm_arm_description): 新增 TCP 链接和 RViz 启动文件

File: src/dm_arm_description/urdf/DM-Arm-Description.urdf (robot description, URDF)
Before this commit: robot TRLC-DK1-Follower, 11 links, 10 joints
Links:
- added link link_tcp
Joints:
- added joint gripper_link_tcp: type fixed, parent link6-7, child link_tcp, origin xyz=0.072 0 0 rpy=-1.5707963267948966 0 -1.5707963267948966
