Commit message: feat(urdf): 新增无夹爪 urdf，修改了关节限制和质量参数

File: description/urdf/dm_arm_no_gripper.urdf (robot description, URDF)
Before this commit: robot DM-Arm, 12 links, 11 joints
Links:
- removed link finger_left
- removed link finger_right
- link link6-7: mass 0.65 -> 0.7
Joints:
- removed joint gripper_left
- removed joint gripper_right
