Commit message: chore: 重构为独立构建的 CMake 项目，作为 dm-arm c++ 核心库，作为机械臂硬件基础平台

File: description/urdf/dm_arm.urdf (robot description, URDF)
Before this commit: robot TRLC-DK1-Follower, 12 links, 11 joints
Links:
- link base_link: geometry collision mesh filename=package://dm_arm_hardware_interface/description/meshes/coll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; visual mesh filename=package://dm_arm_hardware_interface/description/meshes/visu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
- link finger_left: geometry collision mesh filename=package://dm_arm_hardware_interface/description/meshes/coll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; visual mesh filename=package://dm_arm_hardware_interface/description/meshes/visu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
- link finger_right: geometry collision mesh filename=package://dm_arm_hardware_interface/description/meshes/coll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; visual mesh filename=package://dm_arm_hardware_interface/description/meshes/visu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
- link link1-2: geometry collision mesh filename=package://dm_arm_hardware_interface/description/meshes/coll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; visual mesh filename=package://dm_arm_hardware_interface/description/meshes/visu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
- link link2-3: geometry collision mesh filename=package://dm_arm_hardware_interface/description/meshes/coll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; visual mesh filename=package://dm_arm_hardware_interface/description/meshes/visu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
- link link3-4: geometry collision mesh filename=package://dm_arm_hardware_interface/description/meshes/coll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; visual mesh filename=package://dm_arm_hardware_interface/description/meshes/visu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
- link link4-5: geometry collision mesh filename=package://dm_arm_hardware_interface/description/meshes/coll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; visual mesh filename=package://dm_arm_hardware_interface/description/meshes/visu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
- link link5-6: geometry collision mesh filename=package://dm_arm_hardware_interface/description/meshes/coll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; visual mesh filename=package://dm_arm_hardware_interface/description/meshes/visu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
- link link6-7: geometry collision mesh filename=package://dm_arm_hardware_interface/description/meshes/coll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; visual mesh filename=package://dm_arm_hardware_interface/description/meshes/visu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

Commit message: feat(urdf): 标定了夹爪的质量参数

File: description/urdf/dm_arm.urdf (robot description, URDF)
Before this commit: robot DM-Arm, 12 links, 11 joints
Links:
- link finger_left: mass 0.07 -> 0.05
- link finger_right: mass 0.07 -> 0.05
- link link6-7: mass 0.65 -> 0.7
