Commit message: refactor: 重构为 dm_arm_core 包，新增 dm_arm_ros2_control 适配包

File: src/dm_arm_core/description/urdf/dm_arm.urdf (robot description, URDF)
Before this commit: robot DM-Arm, 10 links, 9 joints
Links:
- added link finger_left, mass 0.05; collision mesh filename=package://dm_arm_core/description/meshes/collision/finger_l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; visual mesh filename=package://dm_arm_core/description/meshes/visual/finger_left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
- added link finger_right, mass 0.05; collision mesh filename=package://dm_arm_core/description/meshes/collision/finger_r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; visual mesh filename=package://dm_arm_core/description/meshes/visual/finger_righ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
- link base_link: geometry collision mesh filename=package://dm_arm_core/description/meshes/collision/base_lin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; visual mesh filename=package://dm_arm_core/description/meshes/visual/base_link.g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
- link link1-2: geometry collision mesh filename=package://dm_arm_core/description/meshes/collision/link1-2.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; visual mesh filename=package://dm_arm_core/description/meshes/visual/link1-2.glb
- link link2-3: geometry collision mesh filename=package://dm_arm_core/description/meshes/collision/link2-3.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; visual mesh filename=package://dm_arm_core/description/meshes/visual/link2-3.glb
- link link3-4: geometry collision mesh filename=package://dm_arm_core/description/meshes/collision/link3-4.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; visual mesh filename=package://dm_arm_core/description/meshes/visual/link3-4.glb
- link link4-5: geometry collision mesh filename=package://dm_arm_core/description/meshes/collision/link4-5.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; visual mesh filename=package://dm_arm_core/description/meshes/visual/link4-5.glb
- link link5-6: geometry collision mesh filename=package://dm_arm_core/description/meshes/collision/link5-6.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; visual mesh filename=package://dm_arm_core/description/meshes/visual/link5-6.glb
- link link6-7: geometry collision mesh filename=package://dm_arm_core/description/meshes/collision/link6-7.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; visual mesh filename=package://dm_arm_core/description/meshes/visual/link6-7.glb
Joints:
- added joint gripper_left: type prismatic, parent link6-7, child finger_left, origin xyz=0 0 0 rpy=0 0 0, axis 0 1 0, limit lower=-0.045 upper=0.001 effort=20 velocity=0.18
- added joint gripper_right: type prismatic, parent link6-7, child finger_right, origin xyz=0 0 0 rpy=0 0 0, axis 0 -1 0, limit lower=-0.045 upper=0.001 effort=20 velocity=0.18, mimic joint=gripper_left multiplier=1.0 offset=0.0

File: src/dm_arm_core/description/urdf/dm_arm_no_gripper.urdf (robot description, URDF)
Before this commit: robot DM-Arm, 12 links, 11 joints
Links:
- removed link finger_left
- removed link finger_right
- link base_link: geometry collision mesh filename=package://dm_arm_core/description/meshes/collision/base_lin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; visual mesh filename=package://dm_arm_core/description/meshes/visual/base_link.g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
- link link1-2: geometry collision mesh filename=package://dm_arm_core/description/meshes/collision/link1-2.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; visual mesh filename=package://dm_arm_core/description/meshes/visual/link1-2.glb
- link link2-3: geometry collision mesh filename=package://dm_arm_core/description/meshes/collision/link2-3.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; visual mesh filename=package://dm_arm_core/description/meshes/visual/link2-3.glb
- link link3-4: geometry collision mesh filename=package://dm_arm_core/description/meshes/collision/link3-4.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; visual mesh filename=package://dm_arm_core/description/meshes/visual/link3-4.glb
- link link4-5: geometry collision mesh filename=package://dm_arm_core/description/meshes/collision/link4-5.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; visual mesh filename=package://dm_arm_core/description/meshes/visual/link4-5.glb
- link link5-6: geometry collision mesh filename=package://dm_arm_core/description/meshes/collision/link5-6.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; visual mesh filename=package://dm_arm_core/description/meshes/visual/link5-6.glb
- link link6-7: geometry collision mesh filename=package://dm_arm_core/description/meshes/collision/link6-7.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; visual mesh filename=package://dm_arm_core/description/meshes/visual/link6-7.glb
Joints:
- removed joint gripper_left
- removed joint gripper_right
