Commit message: feat(mock): 新增离线模拟 MotorBus，用于 runtime.write_enabled=false 的后端

File: src/adapters/dm_arm_ros2_control/urdf/dm_arm.ros2_control.xacro (robot description, xacro)
@@ -1,10 +1,9 @@
 <?xml version="1.0"?>
 <robot xmlns:xacro="http://www.ros.org/wiki/xacro">
-  <xacro:macro name="dm_arm_ros2_control" params="name config_file allow_hardware:=false">
+  <xacro:macro name="dm_arm_ros2_control" params="name config_file">
     <ros2_control name="${name}" type="system">
       <hardware>
         <plugin>dm_arm_ros2_control/DmArmSystem</plugin>
         <param name="config_file">${config_file}</param>
-        <param name="allow_hardware">${allow_hardware}</param>
       </hardware>
       <joint name="joint1">

Commit message: feat(ros2): 完善 ros2_control 后端 feat(bringup): 新增桥接层，统一提供 launch 文件和参数接口

File: src/adapters/dm_arm_ros2_control/urdf/dm_arm.ros2_control.xacro (robot description, xacro)
@@ -1,53 +1,8 @@
 <?xml version="1.0"?>
-<robot xmlns:xacro="http://www.ros.org/wiki/xacro">
-  <xacro:macro name="dm_arm_ros2_control" params="name config_file">
-    <ros2_control name="${name}" type="system">
-      <hardware>
-        <plugin>dm_arm_ros2_control/DmArmSystem</plugin>
-        <param name="config_file">${config_file}</param>
-      </hardware>
-      <joint name="joint1">
-        <command_interface name="position"/>
-        <command_interface name="velocity"/>
-        <state_interface name="position"/>
-        <state_interface name="velocity"/>
-        <state_interface name="effort"/>
-      </joint>
-      <joint name="joint2">
-        <command_interface name="position"/>
-        <command_interface name="velocity"/>
-        <state_interface name="position"/>
-        <state_interface name="velocity"/>
-        <state_interface name="effort"/>
-      </joint>
-      <joint name="joint3">
-        <command_interface name="position"/>
-        <command_interface name="velocity"/>
-        <state_interface name="position"/>
-        <state_interface name="velocity"/>
-        <state_interface name="effort"/>
-      </joint>
-      <joint name="joint4">
-        <command_interface name="position"/>
-        <command_interface name="velocity"/>
-        <state_interface name="position"/>
-        <state_interface name="velocity"/>
-        <state_interface name="effort"/>
-      </joint>
-      <joint name="joint5">
-        <command_interface name="position"/>
-        <command_interface name="velocity"/>
-        <state_interface name="position"/>
-        <state_interface name="velocity"/>
-        <state_interface name="effort"/>
-      </joint>
-      <joint name="joint6">
-        <command_interface name="position"/>
-        <command_interface name="velocity"/>
-        <state_interface name="position"/>
-        <state_interface name="velocity"/>
-        <state_interface name="effort"/>
-      </joint>
-    </ros2_control>
-  </xacro:macro>
+<robot xmlns:xacro="http://www.ros.org/wiki/xacro" name="DM-Arm">
+    <xacro:arg name="robot_profile" default="gray"/>
+    <xacro:arg name="config_file" default=""/>
+    <xacro:include filename="$(find dm_arm_description)/urdf/dm_arm.urdf.xacro"/>
+    <xacro:include filename="$(find dm_arm_ros2_control)/urdf/dm_arm_system.ros2_control.xacro"/>
+    <xacro:dm_arm_ros2_control name="dm_arm" config_file="$(arg config_file)"/>
 </robot>

File: src/core/dm_arm_description/urdf/dm_arm.urdf (robot description, URDF)
Before this commit: robot DM-Arm, 12 links, 11 joints
Links:
- link base_link: geometry collision mesh filename=package://dm_arm_description/meshes/collision/base_link.stl; visual mesh filename=package://dm_arm_description/meshes/visual/base_link.glb
- link finger_left: geometry collision mesh filename=package://dm_arm_description/meshes/collision/finger_left.s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; visual mesh filename=package://dm_arm_description/meshes/visual/finger_left.glb
- link finger_right: geometry collision mesh filename=package://dm_arm_description/meshes/collision/finger_right.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; visual mesh filename=package://dm_arm_description/meshes/visual/finger_right.glb
- link link1-2: geometry collision mesh filename=package://dm_arm_description/meshes/collision/link1-2.stl; visual mesh filename=package://dm_arm_description/meshes/visual/link1-2.glb
- link link2-3: geometry collision mesh filename=package://dm_arm_description/meshes/collision/link2-3.stl; visual mesh filename=package://dm_arm_description/meshes/visual/link2-3.glb
- link link3-4: geometry collision mesh filename=package://dm_arm_description/meshes/collision/link3-4.stl; visual mesh filename=package://dm_arm_description/meshes/visual/link3-4.glb
- link link4-5: geometry collision mesh filename=package://dm_arm_description/meshes/collision/link4-5.stl; visual mesh filename=package://dm_arm_description/meshes/visual/link4-5.glb
- link link5-6: geometry collision mesh filename=package://dm_arm_description/meshes/collision/link5-6.stl; visual mesh filename=package://dm_arm_description/meshes/visual/link5-6.glb
- link link6-7: geometry collision mesh filename=package://dm_arm_description/meshes/collision/link6-7.stl; visual mesh filename=package://dm_arm_description/meshes/visual/link6-7.glb

File: src/core/dm_arm_description/urdf/dm_arm_no_gripper.urdf (robot description, URDF)
Before this commit: robot DM-Arm, 10 links, 9 joints
Links:
- link base_link: geometry collision mesh filename=package://dm_arm_description/meshes/collision/base_link.stl; visual mesh filename=package://dm_arm_description/meshes/visual/base_link.glb
- link link1-2: geometry collision mesh filename=package://dm_arm_description/meshes/collision/link1-2.stl; visual mesh filename=package://dm_arm_description/meshes/visual/link1-2.glb
- link link2-3: geometry collision mesh filename=package://dm_arm_description/meshes/collision/link2-3.stl; visual mesh filename=package://dm_arm_description/meshes/visual/link2-3.glb
- link link3-4: geometry collision mesh filename=package://dm_arm_description/meshes/collision/link3-4.stl; visual mesh filename=package://dm_arm_description/meshes/visual/link3-4.glb
- link link4-5: geometry collision mesh filename=package://dm_arm_description/meshes/collision/link4-5.stl; visual mesh filename=package://dm_arm_description/meshes/visual/link4-5.glb
- link link5-6: geometry collision mesh filename=package://dm_arm_description/meshes/collision/link5-6.stl; visual mesh filename=package://dm_arm_description/meshes/visual/link5-6.glb
- link link6-7: geometry collision mesh filename=package://dm_arm_description/meshes/collision/link6-7.stl; visual mesh filename=package://dm_arm_description/meshes/visual/link6-7.glb

File: src/moveit_config/dm_arm_no_gripper/config/DM-Arm.urdf.xacro (robot description, xacro)
@@ -1,9 +1,4 @@
 <?xml version="1.0"?>
 <robot xmlns:xacro="http://www.ros.org/wiki/xacro" name="DM-Arm">
-    <xacro:arg name="initial_positions_file" default="initial_positions.yaml" />
-    <!-- Import DM-Arm urdf file -->
-    <xacro:include filename="$(find dm_arm_core)/description/urdf/dm_arm_no_gripper.urdf" />
-    <!-- Import control_xacro -->
-    <xacro:include filename="DM-Arm.ros2_control.xacro" />
-    <xacro:DM-Arm_ros2_control name="FakeSystem" initial_positions_file="$(arg initial_positions_file)"/>
+    <xacro:include filename="$(find dm_arm_description)/urdf/dm_arm_no_gripper.urdf" />
 </robot>

File: src/moveit_config/dm_arm_with_gripper/config/DM-Arm.urdf.xacro (robot description, xacro)
@@ -1,9 +1,4 @@
 <?xml version="1.0"?>
 <robot xmlns:xacro="http://www.ros.org/wiki/xacro" name="DM-Arm">
-    <xacro:arg name="initial_positions_file" default="initial_positions.yaml" />
-    <!-- Import DM-Arm urdf file -->
-    <xacro:include filename="$(find dm_arm_core)/description/urdf/dm_arm.urdf" />
-    <!-- Import control_xacro -->
-    <xacro:include filename="DM-Arm.ros2_control.xacro" />
-    <xacro:DM-Arm_ros2_control name="FakeSystem" initial_positions_file="$(arg initial_positions_file)"/>
+    <xacro:include filename="$(find dm_arm_description)/urdf/dm_arm.urdf" />
 </robot>
