Commit message: fix(config): 更正路径

File: src/robot_supports/robots/dm_arm/description/model/gray/urdf/dm_arm.ros2_control.xacro (robot description, xacro)
@@ -4,5 +4,5 @@
     <xacro:arg name="hardware_plugin" default=""/>
     <xacro:arg name="hardware_config" default=""/>
-    <xacro:include filename="$(find dm_arm_description)/model/dm_arm_gray/urdf/dm_arm.urdf.xacro"/>
+    <xacro:include filename="$(find dm_arm_description)/model/gray/urdf/dm_arm_no_gripper.urdf"/>
     <xacro:include filename="$(find serial_arm_ros2_control)/urdf/serial_arm_system.ros2_control.xacro"/>
     <ros2_control name="dm_arm" type="system">

File: src/robot_supports/robots/dm_arm/description/model/gray/urdf/dm_arm_no_gripper.urdf (robot description, URDF)
Before this commit: robot DM-Arm, 10 links, 9 joints
Links:
- link base_link: geometry collision mesh filename=package://dm_arm_description/model/gray/meshes/collision/ba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; visual mesh filename=package://dm_arm_description/model/gray/meshes/visual/base_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
- link link1-2: geometry collision mesh filename=package://dm_arm_description/model/gray/meshes/collision/li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; visual mesh filename=package://dm_arm_description/model/gray/meshes/visual/link1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
- link link2-3: geometry collision mesh filename=package://dm_arm_description/model/gray/meshes/collision/li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; visual mesh filename=package://dm_arm_description/model/gray/meshes/visual/link2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
- link link3-4: geometry collision mesh filename=package://dm_arm_description/model/gray/meshes/collision/li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; visual mesh filename=package://dm_arm_description/model/gray/meshes/visual/link3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
- link link4-5: geometry collision mesh filename=package://dm_arm_description/model/gray/meshes/collision/li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; visual mesh filename=package://dm_arm_description/model/gray/meshes/visual/link4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
- link link5-6: geometry collision mesh filename=package://dm_arm_description/model/gray/meshes/collision/li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; visual mesh filename=package://dm_arm_description/model/gray/meshes/visual/link5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
- link link6-7: geometry collision mesh filename=package://dm_arm_description/model/gray/meshes/collision/li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; visual mesh filename=package://dm_arm_description/model/gray/meshes/visual/link6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

File: src/robot_supports/robots/dm_arm/description/model/white/urdf/dm_arm.ros2_control.xacro (robot description, xacro)
@@ -4,5 +4,5 @@
     <xacro:arg name="hardware_plugin" default=""/>
     <xacro:arg name="hardware_config" default=""/>
-    <xacro:include filename="$(find dm_arm_description)/model/dm_arm_white/urdf/dm_arm.urdf.xacro"/>
+    <xacro:include filename="$(find dm_arm_description)/model/white/urdf/dm_arm.urdf"/>
     <xacro:include filename="$(find serial_arm_ros2_control)/urdf/serial_arm_system.ros2_control.xacro"/>
     <ros2_control name="dm_arm" type="system">

File: src/robot_supports/robots/dm_arm/description/model/white/urdf/dm_arm.urdf (robot description, URDF)
Before this commit: robot DM-Arm, 12 links, 11 joints
Links:
- link base_link: geometry collision mesh filename=package://dm_arm_description/model/white/meshes/collision/b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; visual mesh filename=package://dm_arm_description/model/white/meshes/visual/base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
- link finger_left: geometry collision mesh filename=package://dm_arm_description/model/white/meshes/collision/f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; visual mesh filename=package://dm_arm_description/model/white/meshes/visual/fing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
- link finger_right: geometry collision mesh filename=package://dm_arm_description/model/white/meshes/collision/f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; visual mesh filename=package://dm_arm_description/model/white/meshes/visual/fing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
- link link1-2: geometry collision mesh filename=package://dm_arm_description/model/white/meshes/collision/l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; visual mesh filename=package://dm_arm_description/model/white/meshes/visual/link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
- link link2-3: geometry collision mesh filename=package://dm_arm_description/model/white/meshes/collision/l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; visual mesh filename=package://dm_arm_description/model/white/meshes/visual/link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
- link link3-4: geometry collision mesh filename=package://dm_arm_description/model/white/meshes/collision/l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; visual mesh filename=package://dm_arm_description/model/white/meshes/visual/link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
- link link4-5: geometry collision mesh filename=package://dm_arm_description/model/white/meshes/collision/l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; visual mesh filename=package://dm_arm_description/model/white/meshes/visual/link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
- link link5-6: geometry collision mesh filename=package://dm_arm_description/model/white/meshes/collision/l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; visual mesh filename=package://dm_arm_description/model/white/meshes/visual/link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
- link link6-7: geometry collision mesh filename=package://dm_arm_description/model/white/meshes/collision/l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; visual mesh filename=package://dm_arm_description/model/white/meshes/visual/link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

File: src/robot_supports/robots/dm_arm/moveit_config/dm_arm_no_gripper/config/DM-Arm.urdf.xacro (robot description, xacro)
@@ -1,4 +1,4 @@
 <?xml version="1.0"?>
 <robot xmlns:xacro="http://www.ros.org/wiki/xacro" name="DM-Arm">
-    <xacro:include filename="$(find dm_arm_description)/model/dm_arm_gray/urdf/dm_arm_no_gripper.urdf" />
+    <xacro:include filename="$(find dm_arm_description)/model/gray/urdf/dm_arm_no_gripper.urdf" />
 </robot>

File: src/robot_supports/robots/dm_arm/moveit_config/dm_arm_with_gripper/config/DM-Arm.urdf.xacro (robot description, xacro)
@@ -1,4 +1,4 @@
 <?xml version="1.0"?>
 <robot xmlns:xacro="http://www.ros.org/wiki/xacro" name="DM-Arm">
-    <xacro:include filename="$(find dm_arm_description)/model/dm_arm_white/urdf/dm_arm.urdf" />
+    <xacro:include filename="$(find dm_arm_description)/model/white/urdf/dm_arm.urdf" />
 </robot>
